File: power_supply.sch (KiCad schematic (older format))
At the start: 31 parts, among them J1 PWR_MAIN_LINE, J2 PWR_IN_9V_AC, T1 SMPS-24V, T2 220V-9V-1A, U1 LM317, U2 LM337

Commit message: push pull
Parts:
- removed C?: 100n, symbol Device:C
- removed D?: TLC381, symbol Device:Q_TRIAC_A1A2G
- removed Q?: BC817, symbol Device:Q_NPN_BEC
- removed R? (x2): 10k, symbol Device:R_Small
- removed R?: 1k5, symbol Device:R
- removed R?: 330, symbol Device:R
- removed U?: 4N37, Package_DIP:DIP-6_W7.62mm, symbol Isolator:4N37
- added C10, C11: 0.33u/400V, symbol Device:C
- added C12: 330uF, symbol Device:CP
- added D4: ER900, Diode_THT:D_A-405_P7.62mm_Horizontal, symbol Device:DIAC
- added D5: TLC381, Package_TO_SOT_THT:TO-220-3_Horizontal_TabDown, symbol Device:Q_TRIAC_A1A2G
- added D6: SD103BW, Diode_SMD:D_SOD-123, symbol Device:D_Schottky
- added J5: DESOLDER, Connector_Wire:SolderWirePad_1x02_P5.08mm_Drill1.5mm, symbol Connector_Generic:Conn_01x02
- added L1: 330, symbol Device:L
- added Q3: 2SD669, Package_TO_SOT_THT:TO-126-3_Horizontal_TabDown, symbol Device:Q_NPN_ECB
- added Q4: 2SB649, Package_TO_SOT_THT:TO-126-3_Horizontal_TabDown, symbol Device:Q_PNP_ECB
- added R16: 10k, Resistor_THT:R_Axial_DIN0207_L6.3mm_D2.5mm_P10.16mm_Horizontal, symbol Device:R
- added R17: 330k, Resistor_THT:R_Axial_DIN0207_L6.3mm_D2.5mm_P10.16mm_Horizontal, symbol Device:R
- added R18, R20: 4K7, Resistor_SMD:R_0805_2012Metric_Pad1.15x1.40mm_HandSolder, symbol Device:R
- added R19: 100K, Resistor_SMD:R_0805_2012Metric_Pad1.15x1.40mm_HandSolder, symbol Device:R
- added R22: 220, Resistor_SMD:R_0805_2012Metric_Pad1.15x1.40mm_HandSolder, symbol Device:R_Small
- added R24: 330k, Resistor_SMD:R_0805_2012Metric_Pad1.15x1.40mm_HandSolder, symbol Device:R_Small
- added R25: 2k7, Resistor_SMD:R_0805_2012Metric_Pad1.15x1.40mm_HandSolder, symbol Device:R_Small
- added RV1: 200k, Potentiometer_THT:Potentiometer_ACP_CA14-H2,5_Horizontal, symbol Device:R_POT
- added unit 2 of U3
- added unit 3 of U3
- added U8: LT1073, Package_SO:SOIC-8_3.9x4.9mm_P1.27mm, symbol custom:LT1073
- D1, D2: footprint (none) -> Diode_THT:D_DO-15_P10.16mm_Horizontal
- F1: footprint (none) -> Fuse:Fuseholder_Cylinder-5x20mm_Schurter_0031_8201_Horizontal_Open
- F2: renamed from F?; footprint (none) -> Fuse:Fuseholder_Cylinder-5x20mm_Schurter_0031_8201_Horizontal_Open
- J1, J2: footprint (none) -> Connector_Wire:SolderWirePad_1x02_P5.08mm_Drill1.5mm
- R1, R2, R3, R4: footprint (none) -> Resistor_SMD:R_0805_2012Metric_Pad1.15x1.40mm_HandSolder
- R21: renamed from R?; value 2k2 -> 4K7; footprint (none) -> Resistor_SMD:R_0805_2012Metric_Pad1.15x1.40mm_HandSolder
- R23: renamed from R?; value 22k -> 100K; footprint (none) -> Resistor_SMD:R_0805_2012Metric_Pad1.15x1.40mm_HandSolder
- U1: footprint (none) -> Package_TO_SOT_THT:TO-220-3_Vertical
- U3: renamed from U?; footprint (none) -> Package_SO:SOIC-14_3.9x8.7mm_P1.27mm
Connections:
- net labels added: +15V, 240AV+, 240AV-, FIL_CTRL_N, FIL_CTRL_P
- net labels removed: 15AC+, 15AC-, FB_CTRL, Zero_Detect
- wire segments 125 -> 174
- no-connect marks 1 -> 2
Other:
- moved on the sheet: F1, J1, R21, R23, U3A
