File: solder_station_kicad.sch (KiCad schematic (older format))
At the start: 5 parts

Commit message: push pull
Parts:
- added C7, C8, C9: 10n, Capacitor_SMD:C_0805_2012Metric_Pad1.15x1.40mm_HandSolder, symbol Device:C_Small
- added D3: TL431D, Package_SO:SOIC-8_3.9x4.9mm_P1.27mm, symbol Reference_Voltage:TL431D
- added J3: RT_WELLER, symbol Connector_Generic:Conn_01x03
- added J4: VFD dISPLAY, Connector_PinSocket_2.54mm:PinSocket_1x34_P2.54mm_Vertical, symbol Connector_Generic:Conn_01x34
- added P1: ISP, Connector_PinHeader_2.54mm:PinHeader_2x03_P2.54mm_Vertical, symbol custom:ISP
- added Q1: IRF9540, Package_TO_SOT_THT:TO-220-3_Horizontal_TabDown, symbol Device:Q_PMOS_GDS
- added Q2: 2N7002, Package_TO_SOT_SMD:SOT-23, symbol Transistor_FET:2N7002
- added R10, R11, R13, R9: 1k, Resistor_SMD:R_0805_2012Metric_Pad1.15x1.40mm_HandSolder, symbol Device:R_Small
- added R12: 22k, Resistor_SMD:R_0805_2012Metric_Pad1.15x1.40mm_HandSolder, symbol Device:R_Small
- added R14: 33k, Resistor_SMD:R_0805_2012Metric_Pad1.15x1.40mm_HandSolder, symbol Device:R_Small
- added R15: 10K, Resistor_SMD:R_0805_2012Metric_Pad1.15x1.40mm_HandSolder, symbol Device:R_Small
- added R5: 5k6, Resistor_SMD:R_0805_2012Metric_Pad1.15x1.40mm_HandSolder, symbol Device:R_Small
- added R6: 4k7, Resistor_SMD:R_0805_2012Metric_Pad1.15x1.40mm_HandSolder, symbol Device:R_Small
- added R7: 100k, Resistor_SMD:R_0805_2012Metric_Pad1.15x1.40mm_HandSolder, symbol Device:R_Small
- added R8: 2k2, Resistor_SMD:R_0805_2012Metric_Pad1.15x1.40mm_HandSolder, symbol Device:R_Small
- added U4: TLC272, Package_SO:SOIC-8_3.9x4.9mm_P1.27mm, symbol Amplifier_Operational:TLC272
- added U5: LT1007, Package_SO:SOIC-8_3.9x4.9mm_P1.27mm, symbol Amplifier_Operational:LT1012
- added U6: ATMEGA168-20AU, Package_QFP:TQFP-32_7x7mm_P0.8mm, symbol atmel:ATMEGA168-20AU
- added U7: HV5812-SOIC, Housings_SOIC:SOIC-28W_7.5x17.9mm_Pitch1.27mm, symbol custom:HV5812-SOIC
- U3: renamed from U?; footprint (none) -> Package_SO:SOIC-14_3.9x8.7mm_P1.27mm
Connections:
- net labels added: +15V, +24V, 1G, 2G, 3G, 4G, 5G, 6G, 7G, FBA, FBB, GND, MISO, MOSI, RST, S1, S10, S11, S12, S2, S3, S4, S5, S6, S7, S8, S9, SCK, SOLDER, TEMP, a, b, c, d, e, f, g
- wire segments 2 -> 175
- no-connect marks 4 -> 26
Other:
- note added: "3G 20\n 4G 16\n 5G 13\n 6G 8\n 7G 5\n S10 32 °C\n //S11 31 °F\n S12 29 °C\n S8 4 Kolben\n S7 6 Start Stop\n S5 9 Ofen\n S4 4 Glocke"
- note added: "Pin Connection \n7-LT-44Z\n a 28\n b 27\n c 25\n d 24\n e 22\n f 21\n g 19\n 1G 30\n 1G 26\n 2G 23"
