File: solder_station_pwr.sch (KiCad schematic (older format))
At the start: 31 parts, among them J1 PWR_MAIN_LINE, J2 FB_OUT, J3 Conn_01x04, J4 FB_IN, J6 Conn_01x03, Q3 2SD669, T1 RingTrafo_40U, T2 220V-7V5, U2 L7805, U8 LT1073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

Commit message: schematic done
Parts:
- removed D2: SD103BW, Diode_SMD:D_SOD-123, symbol Device:D_Schottky
- removed J4: FB_IN, Connector_PinHeader_2.54mm:PinHeader_1x02_P2.54mm_Vertical, symbol Connector_Generic:Conn_01x02
- removed J6: Conn_01x03, Connector_PinSocket_2.54mm:PinSocket_1x03_P2.54mm_Vertical_SMD_Pin1Left, symbol Connector_Generic:Conn_01x03
- removed Q3: 2SD669, Package_TO_SOT_THT:TO-126-3_Vertical, symbol Device:Q_NPN_ECB
- removed R3: 1k, Resistor_SMD:R_0805_2012Metric_Pad1.15x1.40mm_HandSolder, symbol Device:R_Small
- removed T1: RingTrafo_40U, custom:Transformer_toroid_v_18mm, symbol Device:Transformer_1P_SS
- added C10, C11: 47u, symbol Device:CP
- added C7: 4700p, Capacitor_SMD:C_0805_2012Metric_Pad1.15x1.40mm_HandSolder, symbol Device:C
- added C8, C9: 1u, Capacitor_SMD:C_0805_2012Metric_Pad1.15x1.40mm_HandSolder, symbol Device:C
- added R1, R6, R7: 47k, symbol Device:R
- added R2: 10k, symbol Device:R
- added R3: 22k, symbol Device:R
- added R4, R5: 18, symbol Device:R
- added U1: LM4871, SO08, symbol LM4871:LM4871
Connections:
- net labels removed: FB1, FB2
- wire segments 113 -> 134
- no-connect marks 3 -> 2
Other:
- moved on the sheet: BR1, C1, C12, C2, C3, C4, C5, C6, D6, F1, J1, J2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

Commit message: add lm4871 as filament heater
Parts:
- BR1: symbol custom:BRIGE_RECTIFIER_+a-a -> solder_station_pwr-rescue:BRIGE_RECTIFIER_+a-a-custom
- C10, C11: footprint (none) -> Capacitor_THT:CP_Radial_D5.0mm_P2.50mm
- C7: footprint Capacitor_SMD:C_0805_2012Metric_Pad1.15x1.40mm_HandSolder -> Capacitor_THT:C_Disc_D3.4mm_W2.1mm_P2.50mm
- C8, C9: footprint Capacitor_SMD:C_0805_2012Metric_Pad1.15x1.40mm_HandSolder -> Capacitor_THT:C_Disc_D3.0mm_W2.0mm_P2.50mm
- R1, R2, R3, R4, R5, R6: footprint (none) -> Resistor_SMD:R_0805_2012Metric_Pad1.15x1.40mm_HandSolder
- R7: value 47k -> 4k7; footprint (none) -> Resistor_SMD:R_0805_2012Metric_Pad1.15x1.40mm_HandSolder
- U1: footprint SO08 -> Package_SO:SOIC-8_3.9x4.9mm_P1.27mm; symbol LM4871:LM4871 -> solder_station_pwr-rescue:LM4871-LM4871
- U8: symbol custom:LT1073 -> solder_station_pwr-rescue:LT1073-custom
Connections:
- net +36V: now also J3.1 (Pin_1); no longer J3.4 (Pin_4)
- net +5V: now also J3.2 (Pin_2); no longer J3.1 (Pin_1)
- net -5V: now also J3.4 (Pin_4); no longer J3.3 (Pin_3)
- net GND: now also J3.3 (Pin_3); no longer J3.2 (Pin_2)
Other:
- moved on the sheet: J3
Changed lines of the file:
@@
 EESchema Schematic File Version 4
 LIBS:solder_station_pwr-cache
-EELAYER 29 0
+EELAYER 26 0
 EELAYER END
 $Descr A4 11693 8268
@@
 240AV-
 $Comp
-L custom:LT1073 U8
+L solder_station_pwr-rescue:LT1073-custom U8
 U 1 1 5B3866C0
 P 1900 2350
@@
 	5700 2300 6300 2300
 $Comp
-L custom:BRIGE_RECTIFIER_+a-a BR1
+L solder_station_pwr-rescue:BRIGE_RECTIFIER_+a-a-custom BR1
 U 1 1 5B711570
 P 7850 2800
@@
 L power:+36V #PWR01
 U 1 1 5B5C145A
-P 10350 5400
-F 0 "#PWR01" H 10350 5250 50  0001 C CNN
-F 1 "+36V" H 10365 5573 50  0000 C CNN
-F 2 "" H 10350 5400 50  0001 C CNN
-F 3 "" H 10350 5400 50  0001 C CNN
-	1    10350 5400
+P 10350 5250
+F 0 "#PWR01" H 10350 5100 50  0001 C CNN
+F 1 "+36V" H 10365 5423 50  0000 C CNN
+F 2 "" H 10350 5250 50  0001 C CNN
+F 3 "" H 10350 5250 50  0001 C CNN
+	1    10350 5250
 	1    0    0    -1
 $EndComp
@@
 L power:+5V #PWR0104
 U 1 1 5B64B6CC
-P 10150 5400
-F 0 "#PWR0104" H 10150 5250 50  0001 C CNN
-F 1 "+5V" H 10165 5573 50  0000 C CNN
-F 2 "" H 10150 5400 50  0001 C CNN
-F 3 "" H 10150 5400 50  0001 C CNN
-	1    10150 5400
+P 10150 5250
+F 0 "#PWR0104" H 10150 5100 50  0001 C CNN
+F 1 "+5V" H 10165 5423 50  0000 C CNN
+F 2 "" H 10150 5250 50  0001 C CNN
+F 3 "" H 10150 5250 50  0001 C CNN
+	1    10150 5250
 	1    0    0    -1
 $EndComp
@@
 	9900 5650 10400 5650
 Wire Wire Line
-	10150 5400 10150 5550
-Wire Wire Line
 	10150 5550 10400 5550
 Wire Wire Line
@@
 L Connector_Generic:Conn_01x04 J3
 U 1 1 5B66CCE5
-P 10600 5650
-F 0 "J3" H 10680 5642 50  0000 L CNN
-F 1 "Conn_01x04" H 10680 5551 50  0000 L CNN
-F 2 "Connector_PinSocket_2.54mm:PinSocket_1x04_P2.54mm_Vertical" H 10600 5650 50  0001 C CNN
-F 3 "~" H 10600 5650 50  0001 C CNN
-	1    10600 5650
-	1    0    0    -1
-$EndComp
-Wire Wire Line
-	10350 5400 10350 5850
-Wire Wire Line
-	10350 5850 10400 5850
+P 10600 5550
+F 0 "J3" H 10680 5542 50  0000 L CNN
+F 1 "Conn_01x04" H 10680 5451 50  0000 L CNN
+F 2 "Connector_PinSocket_2.54mm:PinSocket_1x04_P2.54mm_Vertical" H 10600 5550 50  0001 C CNN
+F 3 "~" H 10600 5550 50  0001 C CNN
+	1    10600 5550
+	1    0    0    -1
+$EndComp
+Wire Wire Line
+	10350 5250 10350 5450
 $Comp
 L power:+36V #PWR0107
@@
 	7200 4950 7200 5300
 $Comp
-L LM4871:LM4871 U1
+L solder_station_pwr-rescue:LM4871-LM4871 U1
 U 1 1 5BF1397B
 P 4650 5800
 F 0 "U1" H 4650 5800 50  0000 C CNN
 F 1 "LM4871" H 4650 5800 50  0001 L BNN
-F 2 "SO08" H 4650 5800 50  0001 L BNN
+F 2 "Package_SO:SOIC-8_3.9x4.9mm_P1.27mm" H 4650 5800 50  0001 L BNN
 F 3 "" H 4650 5800 50  0001 L BNN
 F 4 "National Semiconductor" H 4650 5800 50  0001 L BNN "Field4"
@@
 F 0 "C8" H 3350 6200 50  0000 L CNN
 F 1 "1u" H 3300 6100 50  0000 L CNN
-F 2 "Capacitor_SMD:C_0805_2012Metric_Pad1.15x1.40mm_HandSolder" H 3288 6050 50  0001 C CNN
+F 2 "Capacitor_THT:C_Disc_D3.0mm_W2.0mm_P2.50mm" H 3288 6050 50  0001 C CNN
 F 3 "~" H 3250 6200 50  0001 C CNN
 	1    3250 6200
@@
 F 0 "R2" V 3550 5600 50  0000 C CNN
 F 1 "10k" V 3500 5750 50  0000 C CNN
-F 2 "" V 3430 5750 50  0001 C CNN
+F 2 "Resistor_SMD:R_0805_2012Metric_Pad1.15x1.40mm_HandSolder" V 3430 5750 50  0001 C CNN
 F 3 "~" H 3500 5750 50  0001 C CNN
 	1    3500 5750
@@
 F 0 "R3" V 3700 5250 50  0000 C CNN
 F 1 "22k" V 3800 5250 50  0000 C CNN
-F 2 "" V 3730 5250 50  0001 C CNN
+F 2 "Resistor_SMD:R_0805_2012Metric_Pad1.15x1.40mm_HandSolder" V 3730 5250 50  0001 C CNN
 F 3 "~" H 3800 5250 50  0001 C CNN
 	1    3800 5250
@@
 F 0 "R1" V 3150 4800 50  0000 C CNN
 F 1 "47k" V 3250 4800 50  0000 C CNN
-F 2 "" V 3180 4800 50  0001 C CNN
+F 2 "Resistor_SMD:R_0805_2012Metric_Pad1.15x1.40mm_HandSolder" V 3180 4800 50  0001 C CNN
 F 3 "~" H 3250 4800 50  0001 C CNN
 	1    3250 4800
@@
 F 0 "C7" H 2850 6200 50  0000 L CNN
 F 1 "4700p" H 2800 6100 50  0000 L CNN
-F 2 "Capacitor_SMD:C_0805_2012Metric_Pad1.15x1.40mm_HandSolder" H 2788 6050 50  0001 C CNN
+F 2 "Capacitor_THT:C_Disc_D3.4mm_W2.1mm_P2.50mm" H 2788 6050 50  0001 C CNN
 F 3 "~" H 2750 6200 50  0001 C CNN
 	1    2750 6200
@@
 F 0 "C9" H 5115 5196 50  0000 L CNN
 F 1 "1u" H 5115 5105 50  0000 L CNN
-F 2 "Capacitor_SMD:C_0805_2012Metric_Pad1.15x1.40mm_HandSolder" H 5038 5000 50  0001 C CNN
+F 2 "Capacitor_THT:C_Disc_D3.0mm_W2.0mm_P2.50mm" H 5038 5000 50  0001 C CNN
 F 3 "~" H 5000 5150 50  0001 C CNN
 	1    5000 5150
@@
 F 0 "R5" V 5600 5900 50  0000 C CNN
 F 1 "18" V 5700 5900 50  0000 C CNN
-F 2 "" V 5630 5900 50  0001 C CNN
+F 2 "Resistor_SMD:R_0805_2012Metric_Pad1.15x1.40mm_HandSolder" V 5630 5900 50  0001 C CNN
 F 3 "~" H 5700 5900 50  0001 C CNN
 	1    5700 5900
@@
 F 0 "C10" V 6150 5800 50  0000 C CNN
 F 1 "47u" V 6150 5550 50  0000 C CNN
-F 2 "" H 6138 5550 50  0001 C CNN
+F 2 "Capacitor_THT:CP_Radial_D5.0mm_P2.50mm" H 6138 5550 50  0001 C CNN
 F 3 "~" H 6100 5700 50  0001 C CNN
 	1    6100 5700
@@
 F 0 "R4" V 5600 5700 50  0000 C CNN
 F 1 "18" V 5700 5700 50  0000 C CNN
-F 2 "" V 5630 5700 50  0001 C CNN
+F 2 "Resistor_SMD:R_0805_2012Metric_Pad1.15x1.40mm_HandSolder" V 5630 5700 50  0001 C CNN
 F 3 "~" H 5700 5700 50  0001 C CNN
 	1    5700 5700
@@
 F 0 "C11" V 6450 6000 50  0000 C CNN
 F 1 "47u" V 6450 5750 50  0000 C CNN
-F 2 "" H 6438 5750 50  0001 C CNN
+F 2 "Capacitor_THT:CP_Radial_D5.0mm_P2.50mm" H 6438 5750 50  0001 C CNN
 F 3 "~" H 6400 5900 50  0001 C CNN
 	1    6400 5900
@@
 F 0 "R6" V 6300 5300 50  0000 C CNN
 F 1 "47k" V 6400 5300 50  0000 C CNN
-F 2 "" V 6330 5300 50  0001 C CNN
+F 2 "Resistor_SMD:R_0805_2012Metric_Pad1.15x1.40mm_HandSolder" V 6330 5300 50  0001 C CNN
 F 3 "~" H 6400 5300 50  0001 C CNN
 	1    6400 5300
@@
 P 6900 5300
 F 0 "R7" V 6800 5300 50  0000 C CNN
-F 1 "47k" V 6900 5300 50  0000 C CNN
-F 2 "" V 6830 5300 50  0001 C CNN
+F 1 "4k7" V 6900 5300 50  0000 C CNN
+F 2 "Resistor_SMD:R_0805_2012Metric_Pad1.15x1.40mm_HandSolder" V 6830 5300 50  0001 C CNN
 F 3 "~" H 6900 5300 50  0001 C CNN
 	1    6900 5300
@@
 Wire Wire Line
 	6650 5700 6800 5700
+Wire Wire Line
+	10150 5250 10150 5550
+Wire Wire Line
+	10400 5450 10350 5450
 $EndSCHEMATC

Commit message: version
Parts:
- C7: footprint Capacitor_THT:C_Disc_D3.4mm_W2.1mm_P2.50mm -> Capacitor_THT:C_Disc_D4.3mm_W1.9mm_P5.00mm
- C8, C9: footprint Capacitor_THT:C_Disc_D3.0mm_W2.0mm_P2.50mm -> Capacitor_THT:C_Disc_D4.3mm_W1.9mm_P5.00mm
Changed lines of the file:
@@
 EESchema Schematic File Version 4
 LIBS:solder_station_pwr-cache
-EELAYER 26 0
+EELAYER 29 0
 EELAYER END
 $Descr A4 11693 8268
@@
 F 0 "C8" H 3350 6200 50  0000 L CNN
 F 1 "1u" H 3300 6100 50  0000 L CNN
-F 2 "Capacitor_THT:C_Disc_D3.0mm_W2.0mm_P2.50mm" H 3288 6050 50  0001 C CNN
+F 2 "Capacitor_THT:C_Disc_D4.3mm_W1.9mm_P5.00mm" H 3288 6050 50  0001 C CNN
 F 3 "~" H 3250 6200 50  0001 C CNN
 	1    3250 6200
@@
 F 0 "C7" H 2850 6200 50  0000 L CNN
 F 1 "4700p" H 2800 6100 50  0000 L CNN
-F 2 "Capacitor_THT:C_Disc_D3.4mm_W2.1mm_P2.50mm" H 2788 6050 50  0001 C CNN
+F 2 "Capacitor_THT:C_Disc_D4.3mm_W1.9mm_P5.00mm" H 2788 6050 50  0001 C CNN
 F 3 "~" H 2750 6200 50  0001 C CNN
 	1    2750 6200
@@
 F 0 "C9" H 5115 5196 50  0000 L CNN
 F 1 "1u" H 5115 5105 50  0000 L CNN
-F 2 "Capacitor_THT:C_Disc_D3.0mm_W2.0mm_P2.50mm" H 5038 5000 50  0001 C CNN
+F 2 "Capacitor_THT:C_Disc_D4.3mm_W1.9mm_P5.00mm" H 5038 5000 50  0001 C CNN
 F 3 "~" H 5000 5150 50  0001 C CNN
 	1    5000 5150
